File: pcb/kb.kicad_pcb (KiCad board)
At the start: 2 copper layers, 289 x 97 mm, 73 parts, among them J1 S2B-PH-K-S, K1 Gateron_LP_2.0, K10 Gateron_LP_2.0, K11 Gateron_LP_2.0, K12 Gateron_LP_2.0, K13 Gateron_LP_2.0, K14 Gateron_LP_2.0, K15 Gateron_LP_2.0, K16 Gateron_LP_2.0, K17 Gateron_LP_2.0, K18 Gateron_LP_2.0, K19 Gateron_LP_2.0, K2 Gateron_LP_2.0, K20 Gateron_LP_2.0, K21 Gateron_LP_2.0, K22 Gateron_LP_2.0, K23 Gateron_LP_2.0, K24 Gateron_LP_2.0, K25 Gateron_LP_2.0, K26 Gateron_LP_2.0, K27 Gateron_LP_2.0, K28 Gateron_LP_2.0, K29 Gateron_LP_2.0, K3 Gateron_LP_2.0, K30 Gateron_LP_2.0, K31 Gateron_LP_2.0, K32 Gateron_LP_2.0, K33 Gateron_LP_2.0, K34 Gateron_LP_2.0, K35 Gateron_LP_2.0, K36 Gateron_LP_2.0, K37 Gateron_LP_2.0, K38 Gateron_LP_2.0, K39 Gateron_LP_2.0, K4 Gateron_LP_2.0, K40 Gateron_LP_2.0, K41 Gateron_LP_2.0, K42 Gateron_LP_2.0, K43 Gateron_LP_2.0, K44 Gateron_LP_2.0, K45 Gateron_LP_2.0, K46 Gateron_LP_2.0, K47 Gateron_LP_2.0, K48 Gateron_LP_2.0, K49 Gateron_LP_2.0, K5 Gateron_LP_2.0, K50 Gateron_LP_2.0, K51 Gateron_LP_2.0, K52 Gateron_LP_2.0, K53 Gateron_LP_2.0, K54 Gateron_LP_2.0, K55 Gateron_LP_2.0, K56 Gateron_LP_2.0, K57 Gateron_LP_2.0, K58 Gateron_LP_2.0, K59 Gateron_LP_2.0, K6 Gateron_LP_2.0, K60 Gateron_LP_2.0, K61 Gateron_LP_2.0, K62 Gateron_LP_2.0, K63 Gateron_LP_2.0, K64 Gateron_LP_2.0, K7 Gateron_LP_2.0, K8 Gateron_LP_2.0, K9 Gateron_LP_2.0, U1 SuperMini nRF52840

Commit message: use 1/8u pcb grid
Parts:
- removed J1: S2B-PH-K-S, Connector_JST:JST_PH_S2B-PH-K_1x02_P2.00mm_Horizontal
- D1, D2, D3, D4, D5, D6, D7, U1: moved to F.Cu
- moved K56 527.3 mm to (578.4, 164.6)
- moved K57 526.1 mm to (596.8, 48.6)
- moved K42 502.1 mm to (559.9, 65.2)
- moved K58 500.1 mm to (596.8, 65.2)
- moved K43 472.2 mm to (559.9, 81.7)
- moved K44 452.4 mm to (559.9, 98.3)
- moved U1 434.6 mm to (471.9, 191.4), turned to 0 degrees
- moved K45 433.2 mm to (559.9, 114.9)
- moved K59 426.8 mm to (596.8, 81.7)
- moved K31 424.4 mm to (523.0, 148.0)
- moved D3 415.9 mm to (489.2, 181.4), turned to 0 degrees
- moved K46 414.6 mm to (559.9, 131.4)
- moved K32 408.2 mm to (523.0, 164.6)
- moved K33 402.2 mm to (541.5, 48.6)
- moved D4 398.5 mm to (489.2, 184.8), turned to 0 degrees
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Connections:
- U1 pad 1: unconnected-(U1-P0.06-Pad1) -> /ROW1A
- U1 pad 13: Net-(J1-Pin_2) -> unconnected-(U1-BAT+-Pad13)
- U1 pad 2: unconnected-(U1-P0.08-Pad2) -> /ROW1B
- U1 pad 29: Net-(J1-Pin_1) -> unconnected-(U1-BAT+-Pad29)
Routing:
- net Net-(D1-A): track 437.5 -> 0.00 mm
- net Net-(D2-A): track 405.8 -> 0.00 mm
- net Net-(D3-A): track 358.3 -> 0.00 mm
- net Net-(D4-A): track 279.0 -> 0.00 mm
- net /COL1: track 261.1 -> 0.00 mm
- net Net-(D5-A): track 246.5 -> 0.00 mm
- net /COL2: track 229.2 -> 0.00 mm
- net /COL7: track 111.3 -> 0.00 mm
- net Net-(D6-A): track 91.3 -> 0.00 mm
- net /COL6: track 89.5 -> 0.00 mm
- net Net-(D7-A): track 69.2 -> 0.00 mm
- net /COL5: track 67.1 -> 0.00 mm
- net /COL4: track 45.2 -> 0.00 mm
- net /COL3: track 22.0 -> 0.00 mm
- net (no net): vias 16 -> 0
Other:
- board outline removed

Commit message: full layout with 19.05mm spacing
Parts:
- moved K56 542.4 mm to (38.1, 116.7)
- moved K57 541.6 mm to (59.5, 116.7)
- moved K58 518.4 mm to (81.0, 116.7)
- moved K42 515.7 mm to (45.2, 97.6)
- moved K43 486.3 mm to (73.8, 97.6)
- moved K44 467.0 mm to (92.9, 97.6)
- moved K45 448.3 mm to (111.9, 97.6)
- moved K59 443.4 mm to (154.8, 116.7)
- moved K31 440.4 mm to (88.1, 78.6)
- moved K46 430.3 mm to (131.0, 97.6)
- moved K32 424.6 mm to (107.2, 78.6)
- moved K33 416.3 mm to (126.2, 78.6)
- moved K47 413.0 mm to (150.0, 97.6)
- moved K11 400.8 mm to (226.2, 40.5)
- moved K20 400.8 mm to (140.5, 59.5)
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
Commit message: placed all components
Parts:
- added REF**: 6.25U Stabilizer, Gateron_KS33_Hotswap:Gateron-KS33-6.25u-Stabilizer-Cutout, F.Cu at (159.5, 116.7)
- added REF**: 2U Stabilizer, Gateron_KS33_Hotswap:Gateron-KS33-2u-Stabilizer-Cutout, F.Cu at (50.0, 97.6)
- added REF**: 2U Stabilizer, Gateron_KS33_Hotswap:Gateron-KS33-2u-Stabilizer-Cutout, F.Cu at (295.3, 78.6)
- added REF**: 2U Stabilizer, Gateron_KS33_Hotswap:Gateron-KS33-2u-Stabilizer-Cutout, F.Cu at (297.7, 40.5)
- D1, D2, D3, D4, D5, D6, D7, U1: moved to B.Cu
- moved U1 450.6 mm to (46.7, 42.4), turned to -90 degrees
- moved D7 344.7 mm to (181.0, 40.5), turned to -90 degrees
- moved D6 326.3 mm to (200.0, 40.5), turned to -90 degrees
- moved D5 307.9 mm to (219.1, 40.5), turned to -90 degrees
- moved D4 289.6 mm to (238.1, 40.5), turned to -90 degrees
- moved D3 271.5 mm to (257.2, 40.5), turned to -90 degrees
- moved D2 253.6 mm to (276.2, 40.5), turned to -90 degrees
- moved D1 228.1 mm to (304.8, 40.5), turned to -90 degrees
- moved K40 4.76 mm to (264.3, 78.6)
- moved K54 4.76 mm to (288.1, 97.6)
- moved K63 4.76 mm to (288.1, 116.7)
- moved K10 4.76 mm to (211.9, 40.5)
- moved K21 4.76 mm to (164.3, 59.5)
- moved K24 4.76 mm to (221.5, 59.5)
- moved K34 4.76 mm to (150.0, 78.6)
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Other:
- board outline added: 290.5 x 100 mm

Commit message: routed column traces
Connections:
- U1 pad 11: /COL4 -> /COL6
- U1 pad 12: /COL3 -> /COL7
- U1 pad 8: /COL7 -> /COL3
- U1 pad 9: /COL6 -> /COL4
Routing:
- net Net-(D1-A): track 0.00 -> 434.7 mm
- net Net-(D2-A): track 0.00 -> 411.4 mm
- net Net-(D3-A): track 0.00 -> 362.9 mm
- net Net-(D4-A): track 0.00 -> 296.5 mm
- net Net-(D5-A): track 0.00 -> 267.4 mm
- net /COL1: track 0.00 -> 264.9 mm
- net /COL2: track 0.00 -> 232.1 mm
- net Net-(D6-A): track 0.00 -> 215.8 mm
- net /COL3: track 0.00 -> 210.3 mm
- net /COL4: track 0.00 -> 188.3 mm
- net /COL5: track 0.00 -> 166.4 mm
- net Net-(D7-A): track 0.00 -> 155.0 mm
- net /COL6: track 0.00 -> 144.6 mm
- net /COL7: track 0.00 -> 122.0 mm

Commit message: routed all traces
Connections:
- U1 pad 17: unconnected-(U1-P0.31-LF-Pad17) -> /ROW5A
- U1 pad 18: unconnected-(U1-P0.29-LF-Pad18) -> /ROW4A
- U1 pad 19: unconnected-(U1-P0.02-LF-Pad19) -> /ROW3A
- U1 pad 20: unconnected-(U1-P1.15-LF-Pad20) -> /ROW2A
- U1 pad 21: unconnected-(U1-P1.13-LF-Pad21) -> /ROW5B
- U1 pad 22: unconnected-(U1-P1.11-LF-Pad22) -> /ROW4B
- U1 pad 23: unconnected-(U1-P0.10-LF-Pad23) -> /ROW3B
- U1 pad 24: unconnected-(U1-P0.09-LF-Pad24) -> /ROW2B
Routing:
- net /ROW5B: track 0.00 -> 313.3 mm, vias 0 -> 5
- net /ROW4B: track 0.00 -> 309.6 mm, vias 0 -> 7
- net /ROW1B: track 0.00 -> 282.0 mm, vias 0 -> 7
- net /ROW3B: track 0.00 -> 278.3 mm, vias 0 -> 6
- net /ROW2B: track 0.00 -> 270.4 mm, vias 0 -> 7
- net /ROW4A: track 0.00 -> 214.3 mm, vias 0 -> 7
- net /ROW5A: track 0.00 -> 207.0 mm, vias 0 -> 4
- net /ROW3A: track 0.00 -> 187.3 mm, vias 0 -> 7
- net /ROW2A: track 0.00 -> 166.4 mm, vias 0 -> 7
- net /ROW1A: track 0.00 -> 133.9 mm
- net /COL1: track 264.9 -> 266.2 mm

Commit message: tiny fix
Routing:
- net /ROW3A: track 187.3 -> 188.9 mm
- net /COL7: track 122.0 -> 122.7 mm
Changed lines of the file:
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@@
 			(outputformat 1)
 			(mirror no)
-			(drillshape 1)
+			(drillshape 0)
 			(scaleselection 1)
-			(outputdirectory "")
+			(outputdirectory "manufacturing/")
 		)
 	)
@@
 		(descr "Hot Swap Socket for Gateron Low Profile Switch")
 		(property "Reference" "K1"
-			(at 0 9.5 0)
+			(at -4.41325 7.77875 0)
 			(layer "B.SilkS")
 			(effects
@@
 		(descr "Hot Swap Socket for Gateron Low Profile Switch")
 		(property "Reference" "K2"
-			(at 0 9.5 0)
+			(at -4.41325 7.77875 0)
 			(layer "B.SilkS")
 			(effects
@@
 		(sheetfile "kb.kicad_sch")
 		(attr through_hole exclude_from_pos_files exclude_from_bom)
-		(fp_line
-			(start -3.55 14.2)
-			(end -3.55 17.78)
-			(stroke
-				(width 0.15)
-				(type default)
-			)
-			(layer "B.SilkS")
-		)
-		(fp_line
-			(start 3.55 14.2)
-			(end 3.55 17.78)
-			(stroke
-				(width 0.15)
-				(type default)
-			)
-			(layer "B.SilkS")
-		)
-		(fp_line
-			(start 3.55 14.2)
-			(end -3.55 14.2)
-			(stroke
-				(width 0.15)
-				(type default)
-			)
-			(layer "B.SilkS")
-		)
 		(fp_rect
 			(start -8.89 17.78)
@@
 			(layer "Cmts.User")
 		)
-		(fp_text user "topside"
-			(at 0 14.8 90)
-			(unlocked yes)
-			(layer "B.SilkS")
-			(effects
-				(font
-					(size 1 1)
-					(thickness 0.15)
-				)
-				(justify bottom mirror)
-			)
-		)
 		(fp_text user "1"
 			(at -5.715 13.2825 90)
@@
 		(fp_text user "USB"
 			(at 0 16.2 90)
-			(unlocked yes)
-			(layer "B.SilkS")
-			(effects
-				(font
-					(size 1 1)
-					(thickness 0.15)
-				)
-				(justify bottom mirror)
-			)
-		)
-		(fp_text user "USB"
-			(at 0 16.2 90)
 			(layer "Cmts.User")
 			(effects
@@
 	)
 	(segment
-		(start 37.084 63.40475)
-		(end 50.4825 50.00625)
+		(start 37.084 63.5)
+		(end 50.4825 50.1015)
 		(width 0.254)
 		(layer "F.Cu")
@@
 	)
 	(segment
+		(start 50.4825 50.1015)
+		(end 50.4825 50.00625)
+		(width 0.254)
+		(layer "F.Cu")
+		(net 12)
+	)
+	(segment
 		(start 37.084 67.564)
-		(end 37.084 63.40475)
+		(end 37.084 63.5)
 		(width 0.254)
 		(layer "F.Cu")
@@
 	)
 	(segment
+		(start 39.37 86.614)
+		(end 160.782 86.614)
+		(width 0.254)
+		(layer "F.Cu")
+		(net 14)
+	)
+	(segment
 		(start 47.9425 50.00625)
-		(end 36.483 61.46575)
+		(end 47.9425 51.8795)
 		(width 0.2)
 		(layer "F.Cu")
@@
 	)
 	(segment
-		(start 39.37 86.614)
-		(end 160.782 86.614)
-		(width 0.254)
+		(start 34.55625 65.26575)
+		(end 34.55625 81.80025)
+		(width 0.2)
 		(layer "F.Cu")
 		(net 14)
 	)
 	(segment
-		(start 36.483 83.727)
+		(start 34.55625 81.80025)
 		(end 39.37 86.614)
 		(width 0.2)
@@
 	)
 	(segment
-		(start 36.483 61.46575)
-		(end 36.483 83.727)
+		(start 47.9425 51.8795)
+		(end 34.55625 65.26575)
 		(width 0.2)
 		(layer "F.Cu")
@@
 	)
 	(segment
-		(start 34.15525 61.2535)
-		(end 34.15525 104.080192)
+		(start 34.15525 104.080192)
+		(end 35.739058 105.664)
 		(width 0.2)
 		(layer "F.Cu")
@@
 	)
 	(segment
-		(start 34.15525 104.080192)
-		(end 35.739058 105.664)
+		(start 45.4025 53.6575)
+		(end 34.15525 64.90475)
+		(width 0.2)
+		(layer "F.Cu")
+		(net 16)
+	)
+	(segment
+		(start 34.15525 64.90475)
+		(end 34.15525 104.080192)
 		(width 0.2)
 		(layer "F.Cu")
@@
 	(segment
 		(start 45.4025 50.00625)
-		(end 34.15525 61.2535)
+		(end 45.4025 53.6575)
 		(width 0.2)
 		(layer "F.Cu")
@@
 	)
 	(segment
-		(start 34.544 124.714)
-		(end 56.134 124.714)
-		(width 0.254)
+		(start 33.75425 123.92425)
+		(end 34.544 124.714)
+		(width 0.2)
 		(layer "F.Cu")
 		(net 18)
@@
 	(segment
 		(start 42.8625 50.00625)
-		(end 33.75425 59.1145)
+		(end 42.8625 55.4355)
 		(width 0.2)
 		(layer "F.Cu")
@@
 	)
 	(segment
-		(start 33.75425 59.1145)
+		(start 33.75425 64.54375)
 		(end 33.75425 123.92425)
 		(width 0.2)
@@
 	)
 	(segment
+		(start 34.544 124.714)
+		(end 56.134 124.714)
+		(width 0.254)
+		(layer "F.Cu")
+		(net 18)
+	)
+	(segment
 		(start 145.796 124.714)
 		(end 149.098 121.412)
@@
 	)
 	(segment
-		(start 33.75425 123.92425)
-		(end 34.544 124.714)
+		(start 42.8625 55.4355)
+		(end 33.75425 64.54375)
 		(width 0.2)
 		(layer "F.Cu")
@@
 	)
 	(segment
-		(start 250.827 32.48325)
+		(start 250.85575 32.512)
 		(end 257.175 38.83125)
 		(width 0.127)
@@
 	)
 	(segment
-		(start 50.4825 34.76625)
-		(end 52.7655 32.48325)
+		(start 52.73675 32.512)
+		(end 250.85575 32.512)
 		(width 0.127)
 		(layer "B.Cu")
@@
 	)
 	(segment
-		(start 52.7655 32.48325)
-		(end 250.827 32.48325)
+		(start 50.4825 34.76625)
+		(end 52.73675 32.512)
 		(width 0.127)
 		(layer "B.Cu")
@@
 	)
 	(segment
+		(start 61.479 33.92975)
+		(end 176.0735 33.92975)
+		(width 0.127)
+		(layer "B.Cu")
+		(net 26)
+	)
+	(segment
 		(start 60.6425 34.76625)
-		(end 176.91 34.76625)
+		(end 61.479 33.92975)
 		(width 0.127)
 		(layer "B.Cu")
@@
 	)
 	(segment
-		(start 176.91 34.76625)
+		(start 176.0735 33.92975)
 		(end 180.975 38.83125)
 		(width 0.127)

Commit message: use smd headers to mitigate switch collision
Parts:
- added J1: HARWIN_M20-8771346, M20-8771246:HARWIN_M20-8771346, B.Cu at (46.6, 35.6)
- added J2: HARWIN_M20-8771346, M20-8771246:HARWIN_M20-8771346, B.Cu at (46.6, 50.8)
- moved U1 1.44 mm to (47.9, 43.2)
Connections:
- U1 pad 10: /COL5 -> /COL6
- U1 pad 11: /COL6 -> /COL7
- U1 pad 12: /COL7 -> unconnected-(U1-P1.06-LF-Pad12)
- U1 pad 5: unconnected-(U1-P0.17-Pad5) -> /COL1
- U1 pad 6: /COL1 -> /COL2
- U1 pad 7: /COL2 -> /COL3
- U1 pad 8: /COL3 -> /COL4
- U1 pad 9: /COL4 -> /COL5
Routing:
- net /ROW1B: track 282.0 -> 285.6 mm
- net /COL4: track 188.3 -> 191.8 mm
- net /COL6: track 144.6 -> 148.0 mm
- net /COL2: track 232.1 -> 235.5 mm
- net /COL7: track 122.7 -> 126.0 mm
- net /COL5: track 166.4 -> 169.1 mm
- net /COL3: track 210.2 -> 212.8 mm
- net /ROW4B: track 309.6 -> 308.0 mm
- net /ROW5B: track 313.3 -> 311.7 mm
- net /ROW3B: track 278.3 -> 276.8 mm
- net /ROW2B: track 270.4 -> 268.9 mm
- net /COL1: track 266.2 -> 267.3 mm
- net /ROW2A: track 166.4 -> 167.2 mm

Commit message: clean up and add name
Routing:
- net /COL1: track 267.3 -> 276.8 mm
- net /COL7: track 126.0 -> 125.4 mm
Other:
- board text added: "Benson Zhou - Dec 2025"
- board text added: "KB60 V1.0"
