File: pcb/kb.kicad_pcb (KiCad board)
At the start: 2 copper layers, 290.5 x 100 mm, 78 parts, among them J1 HARWIN_M20-8771346, J2 HARWIN_M20-8771346, K1 Gateron_LP_2.0, K10 Gateron_LP_2.0, K11 Gateron_LP_2.0, K12 Gateron_LP_2.0, K13 Gateron_LP_2.0, K14 Gateron_LP_2.0, K15 Gateron_LP_2.0, K16 Gateron_LP_2.0, K17 Gateron_LP_2.0, K18 Gateron_LP_2.0, K19 Gateron_LP_2.0, K2 Gateron_LP_2.0, K20 Gateron_LP_2.0, K21 Gateron_LP_2.0, K22 Gateron_LP_2.0, K23 Gateron_LP_2.0, K24 Gateron_LP_2.0, K25 Gateron_LP_2.0, K26 Gateron_LP_2.0, K27 Gateron_LP_2.0, K28 Gateron_LP_2.0, K29 Gateron_LP_2.0, K3 Gateron_LP_2.0, K30 Gateron_LP_2.0, K31 Gateron_LP_2.0, K32 Gateron_LP_2.0, K33 Gateron_LP_2.0, K34 Gateron_LP_2.0, K35 Gateron_LP_2.0, K36 Gateron_LP_2.0, K37 Gateron_LP_2.0, K38 Gateron_LP_2.0, K39 Gateron_LP_2.0, K4 Gateron_LP_2.0, K40 Gateron_LP_2.0, K41 Gateron_LP_2.0, K42 Gateron_LP_2.0, K43 Gateron_LP_2.0, K44 Gateron_LP_2.0, K45 Gateron_LP_2.0, K46 Gateron_LP_2.0, K47 Gateron_LP_2.0, K48 Gateron_LP_2.0, K49 Gateron_LP_2.0, K5 Gateron_LP_2.0, K50 Gateron_LP_2.0, K51 Gateron_LP_2.0, K52 Gateron_LP_2.0, K53 Gateron_LP_2.0, K54 Gateron_LP_2.0, K55 Gateron_LP_2.0, K56 Gateron_LP_2.0, K57 Gateron_LP_2.0, K58 Gateron_LP_2.0, K59 Gateron_LP_2.0, K6 Gateron_LP_2.0, K60 Gateron_LP_2.0, K61 Gateron_LP_2.0, K62 Gateron_LP_2.0, K63 Gateron_LP_2.0, K64 Gateron_LP_2.0, K7 Gateron_LP_2.0, K8 Gateron_LP_2.0, K9 Gateron_LP_2.0, U1 SuperMini nRF52840

Commit message: change switch reference
Parts:
- renumbered K1 to SW1, K10 to SW10, K11 to SW11, K12 to SW12, K13 to SW13, K14 to SW14, K15 to SW15, K16 to SW16, K17 to SW17, K18 to SW18, K19 to SW19, K2 to SW2, K20 to SW20, K21 to SW21, K22 to SW22, K23 to SW23, K24 to SW24, K25 to SW25, K26 to SW26, K27 to SW27, K28 to SW28, K29 to SW29, K3 to SW3, K30 to SW30, K31 to SW31, K32 to SW32, K33 to SW33, K34 to SW34, K35 to SW35, K36 to SW36, K37 to SW37, K38 to SW38, K39 to SW39, K4 to SW4, K40 to SW40, K41 to SW41, K42 to SW42, K43 to SW43, K44 to SW44, K45 to SW45, K46 to SW46, K47 to SW47, K48 to SW48, K49 to SW49, K5 to SW5, K50 to SW50, K51 to SW51, K52 to SW52, K53 to SW53, K54 to SW54, K55 to SW55, K56 to SW56, K57 to SW57, K58 to SW58, K59 to SW59, K6 to SW6, K60 to SW60, K61 to SW61, K62 to SW62, K63 to SW63, K64 to SW64, K7 to SW7, K8 to SW8, K9 to SW9

Commit message: rewire and fix everything
Parts:
- added D1: 1N4148W, Diode_SMD:D_SOD-123, B.Cu at (52.4, 59.5)
- added D15: 1N4148W, Diode_SMD:D_SOD-123, B.Cu at (54.8, 78.6)
- added D16: 1N4148W, Diode_SMD:D_SOD-123, B.Cu at (81.0, 78.6)
- added D17: 1N4148W, Diode_SMD:D_SOD-123, B.Cu at (100.0, 78.6)
- added D18: 1N4148W, Diode_SMD:D_SOD-123, B.Cu at (119.1, 78.6)
- added D19: 1N4148W, Diode_SMD:D_SOD-123, B.Cu at (138.1, 78.6)
- added D2: 1N4148W, Diode_SMD:D_SOD-123, B.Cu at (76.2, 59.5)
- added D20: 1N4148W, Diode_SMD:D_SOD-123, B.Cu at (157.2, 78.6)
- added D21: 1N4148W, Diode_SMD:D_SOD-123, B.Cu at (176.4, 78.6)
- added D22: 1N4148W, Diode_SMD:D_SOD-123, B.Cu at (190.5, 59.5)
- added D23: 1N4148W, Diode_SMD:D_SOD-123, B.Cu at (209.6, 59.5)
- added D24: 1N4148W, Diode_SMD:D_SOD-123, B.Cu at (228.6, 59.5)
- added D25: 1N4148W, Diode_SMD:D_SOD-123, B.Cu at (247.7, 59.5)
- added D26: 1N4148W, Diode_SMD:D_SOD-123, B.Cu at (266.7, 59.5)
- added D27: 1N4148W, Diode_SMD:D_SOD-123, B.Cu at (285.8, 59.5)
- added D28: 1N4148W, Diode_SMD:D_SOD-123, B.Cu at (309.6, 59.5)
- added D29: 1N4148W, Diode_SMD:D_SOD-123, B.Cu at (57.1, 97.6)
- added D3: 1N4148W, Diode_SMD:D_SOD-123, B.Cu at (95.2, 59.5)
- added D30: 1N4148W, Diode_SMD:D_SOD-123, B.Cu at (85.7, 97.6)
- added D31: 1N4148W, Diode_SMD:D_SOD-123, B.Cu at (104.8, 97.6)
- added D32: 1N4148W, Diode_SMD:D_SOD-123, B.Cu at (123.8, 97.6)
- added D33: 1N4148W, Diode_SMD:D_SOD-123, B.Cu at (142.9, 97.6)
- added D34: 1N4148W, Diode_SMD:D_SOD-123, B.Cu at (161.9, 97.6)
- added D35: 1N4148W, Diode_SMD:D_SOD-123, B.Cu at (181.0, 97.6)
- added D36: 1N4148W, Diode_SMD:D_SOD-123, B.Cu at (195.3, 78.6)
- added D37: 1N4148W, Diode_SMD:D_SOD-123, B.Cu at (214.3, 78.6)
- added D38: 1N4148W, Diode_SMD:D_SOD-123, B.Cu at (233.4, 78.6)
- added D39: 1N4148W, Diode_SMD:D_SOD-123, B.Cu at (252.4, 78.6)
- added D4: 1N4148W, Diode_SMD:D_SOD-123, B.Cu at (114.3, 59.5)
- added D40: 1N4148W, Diode_SMD:D_SOD-123, B.Cu at (271.5, 78.6)
- added D41: 1N4148W, Diode_SMD:D_SOD-123, B.Cu at (302.4, 78.6)
- added D42: 1N4148W, Diode_SMD:D_SOD-123, B.Cu at (50.0, 116.7)
- added D43: 1N4148W, Diode_SMD:D_SOD-123, B.Cu at (71.4, 116.7)
- added D44: 1N4148W, Diode_SMD:D_SOD-123, B.Cu at (92.9, 116.7)
- added D45: 1N4148W, Diode_SMD:D_SOD-123, B.Cu at (123.8, 109.5)
- added D46: 1N4148W, Diode_SMD:D_SOD-123, B.Cu at (142.9, 109.5)
- added D47: 1N4148W, Diode_SMD:D_SOD-123, B.Cu at (166.7, 116.7)
- added D48: 1N4148W, Diode_SMD:D_SOD-123, B.Cu at (200.0, 109.5)
- added D49: 1N4148W, Diode_SMD:D_SOD-123, B.Cu at (200.0, 97.6)
- added D5: 1N4148W, Diode_SMD:D_SOD-123, B.Cu at (133.3, 59.5)
- added D50: 1N4148W, Diode_SMD:D_SOD-123, B.Cu at (219.1, 97.6)
- added D51: 1N4148W, Diode_SMD:D_SOD-123, B.Cu at (238.1, 97.6)
- added D52: 1N4148W, Diode_SMD:D_SOD-123, B.Cu at (257.2, 97.6)
- added D53: 1N4148W, Diode_SMD:D_SOD-123, B.Cu at (276.2, 97.6)
- added D54: 1N4148W, Diode_SMD:D_SOD-123, B.Cu at (295.3, 97.6)
- added D55: 1N4148W, Diode_SMD:D_SOD-123, B.Cu at (314.3, 97.6)
- added D56: 1N4148W, Diode_SMD:D_SOD-123, B.Cu at (173.8, 123.8)
- added D57: 1N4148W, Diode_SMD:D_SOD-123, B.Cu at (173.8, 119.1)
- added D58: 1N4148W, Diode_SMD:D_SOD-123, B.Cu at (173.8, 114.3)
- added D59: 1N4148W, Diode_SMD:D_SOD-123, B.Cu at (219.1, 109.5)
- added D6: 1N4148W, Diode_SMD:D_SOD-123, B.Cu at (152.4, 59.5)
- added D60: 1N4148W, Diode_SMD:D_SOD-123, B.Cu at (238.1, 116.7)
- added D61: 1N4148W, Diode_SMD:D_SOD-123, B.Cu at (257.2, 116.7)
- added D62: 1N4148W, Diode_SMD:D_SOD-123, B.Cu at (276.2, 116.7)
- added D63: 1N4148W, Diode_SMD:D_SOD-123, B.Cu at (295.3, 116.7)
- added D64: 1N4148W, Diode_SMD:D_SOD-123, B.Cu at (314.3, 116.7)
- added D7: 1N4148W, Diode_SMD:D_SOD-123, B.Cu at (171.4, 59.5)
- moved J2 0.13 mm to (46.6, 50.9)
- moved U1 0.13 mm to (47.9, 43.3)
- moved J1 0.13 mm to (46.6, 35.7)
- renumbered D5 to D10, D4 to D11, D3 to D12, D2 to D13, D1 to D14, D7 to D8, D6 to D9
Connections:
- D10 pad 2: Net-(D5-A) -> Net-(D10-A)
- D11 pad 2: Net-(D4-A) -> Net-(D11-A)
- D12 pad 2: Net-(D3-A) -> Net-(D12-A)
- D13 pad 2: Net-(D2-A) -> Net-(D13-A)
- D14 pad 2: Net-(D1-A) -> Net-(D14-A)
- D8 pad 2: Net-(D7-A) -> Net-(D22-K)
- D9 pad 2: Net-(D6-A) -> Net-(D23-K)
- J1 pad 1: (no net) -> unconnected-(U1-GND-Pad28)
- J1 pad 10: (no net) -> /COL5
- J1 pad 11: (no net) -> /COL6
- J1 pad 12: (no net) -> /COL7
- J1 pad 2: (no net) -> /ROW1A
- J1 pad 3: (no net) -> /ROW1B
- J1 pad 4: (no net) -> unconnected-(U1-GND-Pad3)
- J1 pad 6: (no net) -> /COL1
- J1 pad 7: (no net) -> /COL2
- J1 pad 8: (no net) -> /COL3
- J1 pad 9: (no net) -> /COL4
- J2 pad 10: (no net) -> /ROW5B
- J2 pad 11: (no net) -> /ROW4B
- J2 pad 12: (no net) -> /ROW3B
- J2 pad 13: (no net) -> /ROW2B
- J2 pad 3: (no net) -> unconnected-(U1-GND-Pad14)
- J2 pad 4: (no net) -> unconnected-(U1-RST-Pad15)
- J2 pad 5: (no net) -> unconnected-(U1-3V3-Pad16)
- J2 pad 6: (no net) -> /ROW5A
- J2 pad 7: (no net) -> /ROW4A
- J2 pad 8: (no net) -> /ROW3A
- J2 pad 9: (no net) -> /ROW2A
- SW10 pad 2: Net-(D5-A) -> Net-(D10-A)
- SW11 pad 2: Net-(D4-A) -> Net-(D11-A)
- SW12 pad 2: Net-(D3-A) -> Net-(D12-A)
- SW13 pad 2: Net-(D2-A) -> Net-(D13-A)
- SW14 pad 2: Net-(D1-A) -> Net-(D14-A)
- SW15 pad 2: Net-(D1-A) -> Net-(D1-K)
- SW16 pad 2: Net-(D2-A) -> Net-(D16-A)
- SW17 pad 2: Net-(D3-A) -> Net-(D17-A)
- SW18 pad 2: Net-(D4-A) -> Net-(D18-A)
- SW19 pad 2: Net-(D5-A) -> Net-(D19-A)
- SW20 pad 2: Net-(D6-A) -> Net-(D20-A)
- SW21 pad 2: Net-(D7-A) -> Net-(D21-A)
- SW22 pad 2: Net-(D7-A) -> Net-(D22-A)
- SW23 pad 2: Net-(D6-A) -> Net-(D23-A)
- SW24 pad 2: Net-(D5-A) -> Net-(D24-A)
- SW25 pad 2: Net-(D4-A) -> Net-(D25-A)
- SW26 pad 2: Net-(D3-A) -> Net-(D26-A)
- SW27 pad 2: Net-(D2-A) -> Net-(D27-A)
- SW28 pad 2: Net-(D1-A) -> Net-(D28-A)
- SW29 pad 2: Net-(D1-A) -> Net-(D15-K)
- SW30 pad 2: Net-(D2-A) -> Net-(D16-K)
- SW31 pad 2: Net-(D3-A) -> Net-(D17-K)
- SW32 pad 2: Net-(D4-A) -> Net-(D18-K)
- SW33 pad 2: Net-(D5-A) -> Net-(D19-K)
- SW34 pad 2: Net-(D6-A) -> Net-(D20-K)
- SW35 pad 2: Net-(D7-A) -> Net-(D21-K)
- SW36 pad 2: Net-(D7-A) -> Net-(D36-A)
- SW37 pad 2: Net-(D6-A) -> Net-(D37-A)
- SW38 pad 2: Net-(D5-A) -> Net-(D38-A)
- SW39 pad 2: Net-(D4-A) -> Net-(D39-A)
- SW40 pad 2: Net-(D3-A) -> Net-(D40-A)
- SW41 pad 2: Net-(D2-A) -> Net-(D41-A)
- SW42 pad 2: Net-(D1-A) -> Net-(D29-K)
- SW43 pad 2: Net-(D2-A) -> Net-(D30-K)
- SW44 pad 2: Net-(D3-A) -> Net-(D31-K)
- SW45 pad 2: Net-(D4-A) -> Net-(D32-K)
- SW46 pad 2: Net-(D5-A) -> Net-(D33-K)
- SW47 pad 2: Net-(D6-A) -> Net-(D34-K)
- SW48 pad 2: Net-(D7-A) -> Net-(D35-K)
- SW49 pad 2: Net-(D7-A) -> Net-(D48-K)
- SW50 pad 2: Net-(D6-A) -> Net-(D50-A)
- SW51 pad 2: Net-(D5-A) -> Net-(D51-A)
- SW52 pad 2: Net-(D4-A) -> Net-(D52-A)
- SW53 pad 2: Net-(D3-A) -> Net-(D53-A)
- SW54 pad 2: Net-(D2-A) -> Net-(D54-A)
- SW55 pad 2: Net-(D1-A) -> Net-(D55-A)
- SW56 pad 2: Net-(D1-A) -> Net-(D42-K)
- SW57 pad 2: Net-(D2-A) -> Net-(D43-K)
- SW58 pad 2: Net-(D3-A) -> Net-(D44-K)
- SW59 pad 2: Net-(D6-A) -> Net-(D47-K)
- SW60 pad 2: Net-(D5-A) -> Net-(D46-K)
- SW61 pad 2: Net-(D4-A) -> Net-(D45-K)
- SW62 pad 2: Net-(D3-A) -> Net-(D58-K)
- SW63 pad 2: Net-(D2-A) -> Net-(D57-K)
- SW64 pad 2: Net-(D1-A) -> Net-(D56-K)
- SW8 pad 2: Net-(D7-A) -> Net-(D22-K)
- SW9 pad 2: Net-(D6-A) -> Net-(D23-K)
Routing:
- net Net-(D1-A): track 434.7 -> 13.9 mm
- net Net-(D2-A): track 411.4 -> 15.9 mm
- net Net-(D3-A): track 362.9 -> 15.9 mm
- net Net-(D4-A): track 296.5 -> 15.9 mm
- net Net-(D5-A): track 267.4 -> 15.9 mm
- net Net-(D6-A): track 215.8 -> 15.9 mm
- net Net-(D45-K): track 0.00 -> 157.7 mm
- net Net-(D56-K): track 0.00 -> 145.1 mm
- net Net-(D7-A): track 155.0 -> 15.9 mm
- net Net-(D42-K): track 0.00 -> 129.8 mm
- net Net-(D57-K): track 0.00 -> 127.7 mm
- net Net-(D46-K): track 0.00 -> 123.1 mm
- net Net-(D43-K): track 0.00 -> 111.3 mm
- net Net-(D58-K): track 0.00 -> 110.3 mm
- net Net-(D44-K): track 0.00 -> 94.5 mm
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
Commit message: shrink 2u hotswap pads
Parts:
- added J3: S2B-PH-SM4-TB, Connector_JST:JST_PH_S2B-PH-SM4-TB_1x02-1MP_P2.00mm_Horizontal, B.Cu at (69.7, 52.2)
- J1: value HARWIN_M20-8771346 -> S2B-PH-SM4-TB
Connections:
- J1 pad 1: unconnected-(U1-GND-Pad28) -> GND
- J1 pad 4: unconnected-(U1-GND-Pad3) -> GND
- J2 pad 1: (no net) -> Net-(J3-Pin_1)
- J2 pad 2: (no net) -> Net-(J3-Pin_1)
- J2 pad 3: unconnected-(U1-GND-Pad14) -> GND
- U1 pad 13: unconnected-(U1-BAT+-Pad13) -> Net-(J3-Pin_1)
- U1 pad 14: unconnected-(U1-GND-Pad14) -> GND
- U1 pad 28: unconnected-(U1-GND-Pad28) -> GND
- U1 pad 29: unconnected-(U1-BAT+-Pad29) -> Net-(J3-Pin_1)
- U1 pad 3: unconnected-(U1-GND-Pad3) -> GND
- U1 pad 4: unconnected-(U1-GND-Pad4) -> GND
Routing:
- net GND: track 0.00 -> 63.3 mm
- net Net-(J3-Pin_1): track 0.00 -> 41.1 mm

Commit message: add battery connector
Other:
- board text added: "+ -"
Changed lines of the file:
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@@
 		(at 46.609 35.687)
 		(property "Reference" "J1"
-			(at -13.295 4.385 180)
+			(at -15.875 -2.159 180)
 			(layer "B.SilkS")
 			(effects
@@
 		(at 46.609 50.927)
 		(property "Reference" "J2"
-			(at -13.295 4.385 0)
+			(at -15.875 -2.032 0)
 			(layer "B.SilkS")
 			(effects
@@
 		(attr through_hole exclude_from_pos_files exclude_from_bom)
 		(fp_rect
-			(start -8.89 17.78)
-			(end 8.89 -15.24)
-			(stroke
-				(width 0.15)
-				(type solid)
-			)
-			(fill no)
-			(layer "B.SilkS")
-		)
-		(fp_rect
 			(start -3.55 19.3)
 			(end 3.55 14.2)
@@
 		)
 	)
+	(gr_text "+\n-\n"
+		(at 76.962 54.229 0)
+		(layer "B.SilkS")
+		(effects
+			(font
+				(size 1.5 1.5)
+				(thickness 0.3)
+				(bold yes)
+			)
+			(justify left bottom mirror)
+		)
+	)

Commit message: fix bottom row spacing
Parts:
- moved SW58 4.76 mm to (90.5, 116.7)
- moved D44 4.76 mm to (97.6, 116.7)
- moved REF** 2.38 mm to (161.9, 116.7)
- moved SW59 2.38 mm to (161.9, 116.7)
- moved D43 2.38 mm to (73.8, 116.7)
- moved D47 2.38 mm to (169.1, 116.7)
- moved D56 2.38 mm to (176.2, 123.8)
- moved D57 2.38 mm to (176.2, 119.1)
- moved D58 2.38 mm to (176.2, 114.3)
- moved SW57 2.38 mm to (66.7, 116.7)
Routing:
- net /ROW1B: track 285.2 -> 247.4 mm
- net GND: track 63.3 -> 34.8 mm
- net /ROW3A: track 188.6 -> 168.0 mm
- net /ROW2A: track 167.3 -> 147.5 mm
- net /ROW4A: track 214.0 -> 194.4 mm
- net /ROW1A: track 134.3 -> 124.0 mm
- net /COL1: track 276.8 -> 269.9 mm
- net /COL3: track 212.8 -> 206.9 mm
- net /COL2: track 235.5 -> 229.7 mm
- net /COL5: track 169.1 -> 164.1 mm
- net /COL4: track 191.8 -> 186.9 mm
- net /COL7: track 125.4 -> 121.4 mm
- net /COL6: track 148.0 -> 144.0 mm
- net /ROW5B: track 311.7 -> 308.3 mm
- net /ROW4B: track 308.0 -> 305.2 mm
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
Commit message: compact pcb footprint
Parts:
- removed J1: S2B-PH-SM4-TB, M20-8771246:HARWIN_M20-8771346
- removed J2: HARWIN_M20-8771346, M20-8771246:HARWIN_M20-8771346
- moved J3 19.0 mm to (88.7, 52.2)
- moved U1 2.67 mm to (50.5, 43.4)
Routing:
- net GND: track 34.8 -> 86.5 mm
- net /ROW1B: track 247.4 -> 282.5 mm
- net /ROW3A: track 168.0 -> 191.3 mm
- net Net-(J3-Pin_1): track 41.1 -> 63.5 mm
- net /ROW2A: track 147.5 -> 169.7 mm
- net /ROW4A: track 194.4 -> 215.4 mm
- net /ROW1A: track 124.0 -> 135.7 mm
- net /ROW5A: track 205.1 -> 209.9 mm
- net /COL1: track 269.9 -> 274.2 mm
- net /COL3: track 206.9 -> 210.3 mm
- net /COL6: track 144.0 -> 147.2 mm
- net /COL5: track 164.1 -> 166.5 mm
- net Net-(D46-K): track 123.8 -> 121.5 mm
- net /COL2: track 229.7 -> 232.0 mm
- net /COL7: track 121.4 -> 123.3 mm
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Other:
- board size 290.5 x 100 mm -> 285.8 x 97.6 mm

Commit message: fix traces, designators going off pcb
Parts:
- moved REF** 5.14 mm to (157.0, 115.2)

Commit message: checked all tolerances
Parts:
- moved REF** 5.14 mm to (161.9, 116.7)
- renumbered J3 to J1
